Commit message: updated airfly urdf and xacro

File: models/airfly_hexa/urdf/component_snippets.xacro (robot description, xacro)
@@ -185,5 +185,5 @@
             <input_index>0</input_index>
             <input_offset>0</input_offset>
-            <input_scaling>485</input_scaling>
+            <input_scaling>470</input_scaling>
             <zero_position_disarmed>0</zero_position_disarmed>
             <zero_position_armed>100</zero_position_armed>
@@ -193,5 +193,5 @@
             <input_index>1</input_index>
             <input_offset>0</input_offset>
-            <input_scaling>485</input_scaling>
+            <input_scaling>470</input_scaling>
             <zero_position_disarmed>0</zero_position_disarmed>
             <zero_position_armed>100</zero_position_armed>
@@ -201,5 +201,5 @@
             <input_index>2</input_index>
             <input_offset>0</input_offset>
-            <input_scaling>485</input_scaling>
+            <input_scaling>470</input_scaling>
             <zero_position_disarmed>0</zero_position_disarmed>
             <zero_position_armed>100</zero_position_armed>
@@ -209,5 +209,5 @@
             <input_index>3</input_index>
             <input_offset>0</input_offset>
-            <input_scaling>485</input_scaling>
+            <input_scaling>470</input_scaling>
             <zero_position_disarmed>0</zero_position_disarmed>
             <zero_position_armed>100</zero_position_armed>
@@ -217,5 +217,5 @@
             <input_index>4</input_index>
             <input_offset>0</input_offset>
-            <input_scaling>485</input_scaling>
+            <input_scaling>470</input_scaling>
             <zero_position_disarmed>0</zero_position_disarmed>
             <zero_position_armed>100</zero_position_armed>
@@ -225,5 +225,5 @@
             <input_index>5</input_index>
             <input_offset>0</input_offset>
-            <input_scaling>485</input_scaling>
+            <input_scaling>470</input_scaling>
             <zero_position_disarmed>0</zero_position_disarmed>
             <zero_position_armed>100</zero_position_armed>

File: models/airfly_hexa/urdf/hexa.xacro (robot description, xacro)
@@ -8,5 +8,5 @@
   <xacro:property name="mesh_rotor" value="rotor_1.STL" />
   <xacro:property name="mesh_scale_prop" value="1 1 1"/>
-  <xacro:property name="mass" value="140" /> <!-- [kg] -->
+  <xacro:property name="mass" value="95" /> <!-- [kg] -->
   <xacro:property name="body_width" value="1.944514" /> <!-- [m] -->
   <xacro:property name="body_height" value="2.231896" /> <!-- [m] -->
@@ -16,10 +16,10 @@
   <xacro:property name="length_rotor" value="0.02" /> <!-- [m] -->
   <xacro:property name="radius_rotor" value="0.406" /> <!-- [m] -->
-  <xacro:property name="motor_constant" value="12.16582069e-04" /> <!-- [kg.m/s^2] -->
-  <xacro:property name="moment_constant" value="0.05105" /> <!-- [m] -->
+  <xacro:property name="motor_constant" value="12.010474e-04" /> <!-- [kg.m/s^2] -->
+  <xacro:property name="moment_constant" value="0.06" /> <!-- [m] -->
   <xacro:property name="time_constant_up" value="0.0125" /> <!-- [s] -->
   <xacro:property name="time_constant_down" value="0.025" /> <!-- [s] -->
-  <xacro:property name="max_rot_velocity" value="485" /> <!-- [rad/s] -->
-  <xacro:property name="rotor_drag_coefficient" value="0.08531" />
+  <xacro:property name="max_rot_velocity" value="470" /> <!-- [rad/s] -->
+  <xacro:property name="rotor_drag_coefficient" value="1.4" />
   <xacro:property name="rolling_moment_coefficient" value="0.000001" />
   <xacro:property name="color" value="$(arg visual_material)" />
