Commit message: Updated Xacro files and added lidar

File: models/airfly_hexa/urdf/airfly_hexa.urdf (robot description, URDF)
Before this commit: robot airfly_hexa, 9 links, 8 joints
Links:
- added link lidar, mass 0.01; visual mesh filename=package://airfly_hexa/meshes/Lidar_Lite_Laser_Optics.STL scale=0.002 0.002 0.002
- link base_link_inertia: mass 140 -> 95
Joints:
- added joint lidar_joint: type revolute, parent base_link, child lidar, origin xyz=0 0 -0.3625 rpy=0 0 0, axis 0 0 1, limit lower=0 upper=0 effort=0 velocity=0
- joint rotor_0_joint: axis 0 0 -1 -> -0.274688 -0.000308 0.961533
- joint rotor_1_joint: axis 0 0 -1 -> 0.166323 0.000195 0.986071
- joint rotor_2_joint: axis 0 0 -1 -> -0.137623 0.237729 0.961533
- joint rotor_3_joint: axis 0 0 -1 -> -0.08333 0.14394 0.986072
- joint rotor_4_joint: axis 0 0 -1 -> 0.082997 0.144137 0.986071
- joint rotor_5_joint: axis 0 0 -1 -> -0.137066 -0.238047 0.961533

File: models/airfly_hexa/urdf/component_snippets.xacro (robot description, xacro)
@@ -109,4 +109,63 @@
     </gazebo>
   </xacro:macro>
+  <!-- Macro to add a LiDAR. -->
+  <xacro:macro name="lidar_macro"
+    params="link_name parent_link *origin">
+    <link name="${link_name}">
+      <visual>
+        <origin xyz="0 0 0" rpy="0 0 0" />
+        <geometry>
+          <mesh filename="package://airfly_hexa/meshes/Lidar_Lite_Laser_Optics.STL" scale="0.002 0.002 0.002" />
+        </geometry>
+        <material name="white" />
+      </visual>
+      <inertial>
+        <mass value="0.01" />
+        <origin xyz="0 0 0" rpy="0 0 0" />
+        <inertia ixx="2.1733e-6" ixy="0" ixz="0" iyy="2.1733e-6" iyz="0" izz="1.8e-7" />
+      </inertial>
+    </link>
+    <joint name="${link_name}_joint" type="revolute">
+      <xacro:insert_block name="origin" />
+      <parent link="${parent_link}" />
+      <child link="${link_name}" />
+      <axis xyz="0 0 1"/>
+      <limit lower="0" upper="0" effort="0" velocity="0"/>
+    </joint>
+    <gazebo reference="${link_name}">
+      <sensor name="laser" type="ray">
+        <pose>0 0 0 0 1.57079633 0</pose>
+        <ray>
+          <scan>
+            <horizontal>
+              <samples>1</samples>
+              <resolution>1</resolution>
+              <min_angle>-0</min_angle>
+              <max_angle>0</max_angle>
+            </horizontal>
+          </scan>
+          <range>
+            <min>0.06</min> <!-- do not change: use min_distance (below) for realistic behavior (smaller values cause issues) -->
+            <max>35</max>   <!-- do not change: use min_distance (below) for realistic behavior (bigger values cause issues) -->
+            <resolution>0.01</resolution>
+          </range>
+          <noise>
+            <type>gaussian</type>
+            <mean>0.0</mean>
+            <stddev>0.02</stddev>
+          </noise>
+        </ray>
+        <plugin name="LaserPlugin" filename="libgazebo_lidar_plugin.so">
+          <robotNamespace></robotNamespace>
+          <min_distance>0.2</min_distance>
+          <max_distance>15.0</max_distance>
+        </plugin>
+        <always_on>1</always_on>
+        <update_rate>20</update_rate>
+        <visualize>true</visualize>
+      </sensor>
+      <material>Gazebo/White</material>
+    </gazebo>
+  </xacro:macro>
   <!-- Macro to add the gps_plugin. -->
   <xacro:macro name="gps_plugin_macro" params="namespace gps_noise">

File: models/airfly_hexa/urdf/hexa.xacro (robot description, xacro)
@@ -3,5 +3,5 @@
   <!-- Properties -->
   <xacro:property name="namespace" value="" />
-  <xacro:property name="rotor_velocity_slowdown_sim" value="10" />
+  <xacro:property name="rotor_velocity_slowdown_sim" value="3" />
   <xacro:property name="mesh_file" value="base_link.STL" />
   <xacro:property name="mesh_scale" value="1 1 1"/>
@@ -21,6 +21,6 @@
   <xacro:property name="time_constant_down" value="0.025" /> <!-- [s] -->
   <xacro:property name="max_rot_velocity" value="470" /> <!-- [rad/s] -->
-  <xacro:property name="rotor_drag_coefficient" value="1.4" />
-  <xacro:property name="rolling_moment_coefficient" value="0.000001" />
+  <xacro:property name="rotor_drag_coefficient" value="0.002557889" />
+  <xacro:property name="rolling_moment_coefficient" value="3.172e-06" />
   <xacro:property name="color" value="$(arg visual_material)" />
   <xacro:property name="color_blue" value="BlueTransparent" />
@@ -99,5 +99,5 @@
     <xacro:insert_block name="body_inertia" />
   </xacro:multirotor_base_macro>
-  <!-- Instantiate rotor 4 -->
+  <!-- Instantiate rotor 4 rpy="0.167 -0.005845 2.6538" -->
   <xacro:vertical_rotor
     robot_namespace="${namespace}"
@@ -121,6 +121,7 @@
     <origin xyz="0.85004 -0.42999 0.25919" rpy="0.167 -0.005845 2.6538" />
     <xacro:insert_block name="rotor_inertia_1" />
-  </xacro:vertical_rotor>
-  <!-- Instantiate rotor 5 -->
+    <axis xyz="0.082997 0.144137 0.986071" />
+  </xacro:vertical_rotor>
+  <!-- Instantiate rotor 5 rpy="-0.24255 0.13775 -0.01577" -->
   <xacro:vertical_rotor
     robot_namespace="${namespace}"
@@ -144,6 +145,7 @@
     <origin xyz="-0.78182 0.54846 0.25157" rpy="-0.24255 0.13775 -0.01577" />
     <xacro:insert_block name="rotor_inertia_4" />
-  </xacro:vertical_rotor>
-  <!-- Instantiate rotor 2 -->
+    <axis xyz="-0.137066 -0.238047 0.961533" />
+  </xacro:vertical_rotor>
+  <!-- Instantiate rotor 2 rpy="0.24252 0.13781 0.017864" -->
   <xacro:vertical_rotor robot_namespace="${namespace}"
     suffix="front_left"
@@ -166,6 +168,7 @@
     <origin xyz="0.8659 0.40285 0.25157" rpy="0.24252 0.13781 0.017864" />
     <xacro:insert_block name="rotor_inertia_0" />
-  </xacro:vertical_rotor>
-  <!-- Instantiate rotor 3 -->
+    <axis xyz="-0.137623 0.237729 0.961533" />
+  </xacro:vertical_rotor>
+  <!-- Instantiate rotor 3 rpy="0.14504 0.083268 0.0071482" -->
   <xacro:vertical_rotor robot_namespace="${namespace}"
     suffix="back_right"
@@ -188,6 +191,7 @@
     <origin xyz="-0.7974 -0.52116 0.25919" rpy="0.14504 0.083268 0.0071482" />
     <xacro:insert_block name="rotor_inertia_3" />
-  </xacro:vertical_rotor>
-  <!-- Instantiate rotor 0 -->
+    <axis xyz="-0.08333 0.14394 0.986072" />
+  </xacro:vertical_rotor>
+  <!-- Instantiate rotor 0 rpy="-0.0029981 0.27825 3.1318" -->
   <xacro:vertical_rotor robot_namespace="${namespace}"
     suffix="back_left"
@@ -210,6 +214,7 @@
     <origin xyz="-0.084071 -0.95131 0.25157" rpy="-0.0029981 0.27825 3.1318" />
     <xacro:insert_block name="rotor_inertia_2" />
-  </xacro:vertical_rotor>
-  <!-- Instantiate rotor 1 -->
+    <axis xyz="-0.274688 -0.000308 0.961533" />
+  </xacro:vertical_rotor>
+  <!-- Instantiate rotor 1 rpy="-2.5657e-05 -0.1671 0.0013258" -->
   <xacro:vertical_rotor robot_namespace="${namespace}"
     suffix="back_right"
@@ -232,4 +237,5 @@
     <origin xyz="-0.052635 0.95115 0.25919" rpy="-2.5657e-05 -0.1671 0.0013258" />
     <xacro:insert_block name="rotor_inertia_5" />
+    <axis xyz="0.166323 0.000195 0.986071" />
   </xacro:vertical_rotor>
 </robot>

File: models/airfly_hexa/urdf/hexa_base.xacro (robot description, xacro)
@@ -19,5 +19,5 @@
   <xacro:arg name='send_vision_estimation' default='true' />
   <xacro:arg name='send_odometry' default='false' />
-  <xacro:arg name='enable_lockstep' default='true' />
+  <xacro:arg name='enable_lockstep' default='false' />
   <xacro:arg name='use_tcp' default='true' />
   <xacro:arg name='vehicle_is_tailsitter' default='false' />
@@ -27,4 +27,5 @@
   <!-- The following causes segfault with multiple vehicles if defaults to true!!! -->
   <xacro:arg name='enable_ground_truth' default='false' />
+  <xacro:arg name='enable_lidar' default='false' />
   <xacro:arg name='enable_logging' default='false' />
   <xacro:arg name='log_file' default='airfly_hexa' />
@@ -116,4 +117,14 @@
     <origin xyz="0 0 0" rpy="0 0 0" />
   </xacro:imu_plugin_macro>
+  <!-- Enable LiDAR -->
+  <xacro:if value="$(arg enable_lidar)">
+    <!-- Instantiate LiDAR plugin -->
+    <xacro:lidar_macro
+      link_name="lidar"
+      parent_link="base_link"
+      >
+      <origin xyz="0 0 -0.3625" rpy="0 0 0" />
+    </xacro:lidar_macro>
+  </xacro:if>
   <!-- Enable GroundTruth -->
   <xacro:if value="$(arg enable_ground_truth)">
@@ -122,5 +133,5 @@
       base="base_link"
       pub_rate="30"
-      groundt_topic="/odom"
+      groundt_topic="/ground_truth"
       z_offset = "-0.1975016"
     >

File: models/airfly_hexa/urdf/multirotor_base.xacro (robot description, xacro)
@@ -79,8 +79,8 @@
   <!-- Rotor joint and link -->
   <xacro:macro name="vertical_rotor"
-    params="robot_namespace suffix direction motor_constant moment_constant parent mass_rotor length_rotor radius_rotor time_constant_up time_constant_down max_rot_velocity motor_number rotor_drag_coefficient rolling_moment_coefficient color mesh mesh_scale *origin *inertia">
+    params="robot_namespace suffix direction motor_constant moment_constant parent mass_rotor length_rotor radius_rotor time_constant_up time_constant_down max_rot_velocity motor_number rotor_drag_coefficient rolling_moment_coefficient color mesh mesh_scale *origin *inertia *axis">
     <joint name="rotor_${motor_number}_joint" type="continuous">
       <xacro:insert_block name="origin" />
-      <axis xyz="0 0 -1" />
+      <xacro:insert_block name="axis" />
       <parent link="${parent}" />
       <child link="rotor_${motor_number}" />

Commit message: Updated URDF files with a workable lidar sensor

File: models/airfly_hexa/urdf/airfly_hexa.urdf (robot description, URDF)
Before this commit: robot airfly_hexa, 10 links, 9 joints
Links:
- removed link lidar
- added link lidar_lite::link, mass 0.01; visual mesh filename=package://airfly_hexa/meshes/Lidar_Lite_Laser_Optics.STL scale=0.002 0.002 0.002
Joints:
- joint lidar_joint: child lidar -> lidar_lite::link; origin xyz=0 0 -0.3625 rpy=0 0 0 -> xyz=0 0 -0.36 rpy=0 0 0

File: models/airfly_hexa/urdf/component_snippets.xacro (robot description, xacro)
@@ -126,5 +126,5 @@
       </inertial>
     </link>
-    <joint name="${link_name}_joint" type="revolute">
+    <joint name="lidar_joint" type="revolute">
       <xacro:insert_block name="origin" />
       <parent link="${parent_link}" />
@@ -135,5 +135,5 @@
     <gazebo reference="${link_name}">
       <sensor name="laser" type="ray">
-        <pose>0 0 0 0 1.57079633 0</pose>
+        <pose>0 0 -0.21 0 1.57079633 0</pose>
         <ray>
           <scan>
@@ -156,8 +156,8 @@
           </noise>
         </ray>
-        <plugin name="LaserPlugin" filename="libgazebo_lidar_plugin.so">
+        <plugin name="LaserLitePlugin" filename="libgazebo_lidar_lite_plugin.so">
           <robotNamespace></robotNamespace>
-          <min_distance>0.2</min_distance>
-          <max_distance>15.0</max_distance>
+          <min_distance>0.08</min_distance>
+          <max_distance>30.0</max_distance>
         </plugin>
         <always_on>1</always_on>

File: models/airfly_hexa/urdf/hexa_base.xacro (robot description, xacro)
@@ -121,8 +121,8 @@
     <!-- Instantiate LiDAR plugin -->
     <xacro:lidar_macro
-      link_name="lidar"
+      link_name="lidar_lite::link"
       parent_link="base_link"
       >
-      <origin xyz="0 0 -0.3625" rpy="0 0 0" />
+      <origin xyz="0 0 -0.36" rpy="0 0 0" />
     </xacro:lidar_macro>
   </xacro:if>
